File: Embodiment_01/Lightint_Elefant/LED_Center/LED_Center_001/LED_L_Arm_001.kicad_pcb (KiCad board)
At the start: 2 copper layers, 24 parts, among them J1 Conn_01x01_Female, J10 Conn_01x01_Female, J11 Conn_01x01_Female, J12 Conn_01x01_Female, J2 Conn_01x01_Female, J3 Conn_01x01_Female, J4 Conn_01x01_Female, J5 Conn_01x01_Female, J6 Conn_01x01_Female, J7 Conn_01x01_Female, J8 Conn_01x01_Female, J9 Conn_01x01_Female

Commit message: elefant wings added
Parts:
- moved C1 34.0 mm to (27.2, 20.2)
- moved C2 34.0 mm to (29.5, 35.1)
- moved C3 34.0 mm to (31.7, 20.2)
- moved C4 34.0 mm to (27.2, 23.2)
- moved R1 34.0 mm to (20.2, 35.1)
- moved R2 34.0 mm to (24.9, 35.1)
